Commit message: Complete Assignment 5: Add joint inertia, configure MoveIt settings, and generate flattened URDF

File: src/d11115810_ros2summercamp/urdf/robot.urdf (robot description, URDF)
Before this commit: robot manipulator_robot, 7 links, 6 joints
Links:
- link base_link: mass None -> 2.0
- link gripper_base: mass None -> 0.5
- link left_finger: mass None -> 0.1
- link link_1: mass None -> 1.0
- link link_2: mass None -> 1.0
- link link_3: mass None -> 1.0
- link right_finger: mass None -> 0.1

Commit message: add d11115810_gazebo

File: src/d11115810_ros2summercamp/urdf/robot.urdf (robot description, URDF)
Before this commit: robot manipulator_robot, 7 links, 6 joints
Links:
- added link world
Joints:
- added joint world_to_base_joint: type fixed, parent world, child base_link, origin xyz=0 0 0.15 rpy=0 0 0
